Commit message: adjusting joint 4 + 5 length - macro xacro

File: urdf/abb_irb4600_40_255_macro.xacro (robot description, xacro)
@@ -163,5 +163,5 @@
       <parent link="${prefix}link_3"/>
       <child link="${prefix}link_4"/>
-      <origin xyz="0.332 0 0.175" rpy="0 0 0 "/>
+      <origin xyz="0.331 0 0.175" rpy="0 0 0 "/>
       <axis xyz="1 0 0"/>
       <!-- (-400 to 400) -->
